File: hardware/pcb/hestia/buck_converter.kicad_sch (KiCad schematic)
At the start: 21 parts

Commit message: add mouser number for FB
Parts:
- C1, C23, C26, C33, C36, C37, C4: value (none) -> 47uF 10V
- C2: value (none) -> 4.7nF
- C3, C39: value (none) -> 100p
- C34, C35: value (none) -> 0.1uF
- C38: value (none) -> 2.2n
- C8: value (none) -> 22uF 16V
- D6: value (none) -> FSV330AF
- FB2: value (none) -> 74279220321; Mouser Part (none) -> 810-MPZ2012S331AT000
- L2: value (none) -> 10uH
- R1: value (none) -> 33K
- R20: value (none) -> 0R
- TP2: value (none) -> TestPoint
- U1: value (none) -> LM2655MTC-3.3/NOPB
Changed lines of the file:
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@@
       (effects (font (size 1.27 1.27)) (justify left))
     )
-    (property "Value" "" (id 1) (at 146.685 86.995 0)
+    (property "Value" "LM2655MTC-3.3/NOPB" (id 1) (at 146.685 86.995 0)
       (effects (font (size 0.9 0.9)) (justify left))
     )
@@
     (in_bom yes) (on_board yes)
     (property "Reference" "L2" (id 0) (at 176.53 88.265 90))
-    (property "Value" "" (id 1) (at 177.8 92.075 90))
+    (property "Value" "10uH" (id 1) (at 177.8 92.075 90))
     (property "Footprint" "" (id 2) (at 179.07 90.805 0)
       (effects (font (size 1.27 1.27)) hide)
@@
       (effects (font (size 1.27 1.27)) (justify left))
     )
-    (property "Value" "" (id 1) (at 78.74 96.52 0)
+    (property "Value" "22uF 16V" (id 1) (at 78.74 96.52 0)
       (effects (font (size 1.27 1.27)) (justify left))
     )
@@
       (effects (font (size 1.27 1.27)) (justify right))
     )
-    (property "Value" "" (id 1) (at 120.015 93.345 0)
+    (property "Value" "0.1uF" (id 1) (at 120.015 93.345 0)
       (effects (font (size 1.27 1.27)) (justify right))
     )
@@
     (in_bom yes) (on_board yes)
     (property "Reference" "TP2" (id 0) (at 212.725 74.295 90))
-    (property "Value" "" (id 1) (at 212.725 80.645 90))
+    (property "Value" "TestPoint" (id 1) (at 212.725 80.645 90))
     (property "Footprint" "" (id 2) (at 217.805 89.535 0)
       (effects (font (size 1.27 1.27)) hide)
@@
     (in_bom yes) (on_board yes)
     (property "Reference" "C38" (id 0) (at 117.475 66.675 90))
-    (property "Value" "" (id 1) (at 117.475 69.215 90))
+    (property "Value" "2.2n" (id 1) (at 117.475 69.215 90))
     (property "Footprint" "" (id 2) (at 117.475 71.4502 0)
       (effects (font (size 1.27 1.27)) hide)
@@
       (effects (font (size 1.27 1.27)) (justify left))
     )
-    (property "Value" "" (id 1) (at 94.615 95.885 0)
+    (property "Value" "47uF 10V" (id 1) (at 94.615 95.885 0)
       (effects (font (size 1.27 1.27)) (justify left))
     )
@@
       (effects (font (size 1.27 1.27)) (justify left))
     )
-    (property "Value" "" (id 1) (at 162.56 97.79 90)
+    (property "Value" "FSV330AF" (id 1) (at 162.56 97.79 90)
       (effects (font (size 1.27 1.27)) (justify left))
     )
@@
       (effects (font (size 1.27 1.27)) (justify left))
     )
-    (property "Value" "" (id 1) (at 177.8 76.8349 0)
+    (property "Value" "0.1uF" (id 1) (at 177.8 76.8349 0)
       (effects (font (size 1.27 1.27)) (justify left))
     )
@@
       (effects (font (size 1.27 1.27)) (justify left))
     )
-    (property "Value" "" (id 1) (at 100.965 93.345 0)
+    (property "Value" "47uF 10V" (id 1) (at 100.965 93.345 0)
       (effects (font (size 1.27 1.27)) (justify left))
     )
@@
     (in_bom yes) (on_board yes)
     (property "Reference" "R1" (id 0) (at 131.445 65.405 90))
-    (property "Value" "" (id 1) (at 131.445 67.945 90))
+    (property "Value" "33K" (id 1) (at 131.445 67.945 90))
     (property "Footprint" "" (id 2) (at 131.445 68.707 90)
       (effects (font (size 1.27 1.27)) hide)
@@
       (effects (font (size 1.27 1.27)) (justify left))
     )
-    (property "Value" "" (id 1) (at 206.375 93.345 90)
+    (property "Value" "0R" (id 1) (at 206.375 93.345 90)
       (effects (font (size 1.27 1.27)) (justify left))
     )
@@
       (effects (font (size 1.27 1.27)) (justify left))
     )
-    (property "Value" "" (id 1) (at 194.945 104.14 0)
+    (property "Value" "47uF 10V" (id 1) (at 194.945 104.14 0)
       (effects (font (size 1.27 1.27)) (justify left))
     )
@@
       (effects (font (size 1.27 1.27)) (justify left))
     )
-    (property "Value" "" (id 1) (at 88.265 93.345 0)
+    (property "Value" "47uF 10V" (id 1) (at 88.265 93.345 0)
       (effects (font (size 1.27 1.27)) (justify left))
     )
@@
     (in_bom yes) (on_board yes) (fields_autoplaced)
     (property "Reference" "FB2" (id 0) (at 84.4042 78.105 90))
-    (property "Value" "" (id 1) (at 84.4042 80.645 90))
+    (property "Value" "74279220321" (id 1) (at 84.4042 80.645 90))
     (property "Footprint" "" (id 2) (at 84.455 87.503 90)
       (effects (font (size 1.27 1.27)) hide)
@@
     )
     (property "Digikey Part" "732-6125-1-ND" (id 5) (at 84.455 85.725 90)
+      (effects (font (size 1.27 1.27)) hide)
+    )
+    (property "Mouser Part" "810-MPZ2012S331AT000" (id 6) (at 84.455 85.725 0)
       (effects (font (size 1.27 1.27)) hide)
     )
@@
       (effects (font (size 1.27 1.27)) (justify left))
     )
-    (property "Value" "" (id 1) (at 187.96 102.235 0)
+    (property "Value" "47uF 10V" (id 1) (at 187.96 102.235 0)
       (effects (font (size 1.27 1.27)) (justify left))
     )
@@
       (effects (font (size 1.27 1.27)) (justify left))
     )
-    (property "Value" "" (id 1) (at 201.93 102.235 0)
+    (property "Value" "47uF 10V" (id 1) (at 201.93 102.235 0)
       (effects (font (size 1.27 1.27)) (justify left))
     )
@@
     (in_bom yes) (on_board yes)
     (property "Reference" "C39" (id 0) (at 117.475 75.565 90))
-    (property "Value" "" (id 1) (at 117.475 78.105 90))
+    (property "Value" "100p" (id 1) (at 117.475 78.105 90))
     (property "Footprint" "" (id 2) (at 117.475 77.8002 0)
       (effects (font (size 1.27 1.27)) hide)
@@
       (effects (font (size 1.27 1.27)) (justify left))
     )
-    (property "Value" "" (id 1) (at 159.385 117.4749 0)
+    (property "Value" "4.7nF" (id 1) (at 159.385 117.4749 0)
       (effects (font (size 1.27 1.27)) (justify left))
     )
@@
       (effects (font (size 1.27 1.27)) (justify right))
     )
-    (property "Value" "" (id 1) (at 136.525 111.1249 0)
+    (property "Value" "100p" (id 1) (at 136.525 111.1249 0)
       (effects (font (size 1.27 1.27)) (justify right))
     )
@@
       (effects (font (size 1.27 1.27)) (justify left))
     )
-    (property "Value" "" (id 1) (at 107.315 95.885 0)
-      (effects (font (size 1.27 1.27)) (justify left))
-    )
+    (property "Value" "47uF 10V" (id 1) (at 107.315 95.885 0)
+      (effects (font (size 1.27 1.27)) (justify left))
+    )
