File: hardware/pcb/hestia/heater.kicad_sch (KiCad schematic)
At the start: 22 parts, among them Q1 FDS8876, SW2 SW_Push_Open, U10 INA826

Commit message: change d6? to SK34A-LTP with a DO-214AC (SMA) footprint. This diode is a higher profile and may violate height restrictions for some close stacked payload configurations.
Parts:
- C5, C6, C7: footprint (none) -> Capacitor_SMD:C_1206_3216Metric
- C57: footprint (none) -> Capacitor_SMD:C_0603_1608Metric_Pad1.08x0.95mm_HandSolder
- D5: footprint (none) -> LED_SMD:LED_0805_2012Metric_Pad1.15x1.40mm_HandSolder
- D7: footprint (none) -> Package_TO_SOT_SMD:SOT-23
- FB13, R17, R18, R19, R2, R25, R3, R41, R44: footprint (none) -> Resistor_SMD:R_0603_1608Metric_Pad0.98x0.95mm_HandSolder
- Q1: footprint (none) -> Package_SO:SOIC-8_3.9x4.9mm_P1.27mm
- R26: footprint (none) -> NetTie:NetTie-2_SMD_Pad0.5mm
- R42: footprint (none) -> Capacitor_SMD:C_0402_1005Metric
- R43: footprint (none) -> Hestia:LVK12R010CER
- SW2: footprint (none) -> Connector_PinHeader_2.54mm:PinHeader_1x02_P2.54mm_Vertical
- TP1: footprint (none) -> TestPoint:TestPoint_Pad_2.0x2.0mm
- U10: footprint (none) -> Package_SON:WSON-8-1EP_3x3mm_P0.5mm_EP1.2x2mm
Changed lines of the file:
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@@
       (effects (font (size 1.27 1.27)) (justify left))
     )
-    (property "Footprint" "" (id 2) (at 127.762 97.155 90)
+    (property "Footprint" "NetTie:NetTie-2_SMD_Pad0.5mm" (id 2) (at 127.762 97.155 90)
       (effects (font (size 1.27 1.27)) hide)
     )
@@
     (property "Reference" "U10" (id 0) (at 116.205 70.7136 90))
     (property "Value" "INA826" (id 1) (at 116.205 73.2536 90))
-    (property "Footprint" "" (id 2) (at 103.505 76.835 0)
+    (property "Footprint" "Package_SON:WSON-8-1EP_3x3mm_P0.5mm_EP1.2x2mm" (id 2) (at 103.505 76.835 0)
       (effects (font (size 1.27 1.27)) hide)
     )
@@
     (property "Reference" "R2" (id 0) (at 106.045 116.205 90))
     (property "Value" "470R" (id 1) (at 106.045 118.745 90))
-    (property "Footprint" "" (id 2) (at 106.045 124.333 90)
+    (property "Footprint" "Resistor_SMD:R_0603_1608Metric_Pad0.98x0.95mm_HandSolder" (id 2) (at 106.045 124.333 90)
       (effects (font (size 1.27 1.27)) hide)
     )
@@
       (effects (font (size 1.27 1.27)) (justify right))
     )
-    (property "Footprint" "" (id 2) (at 100.965 137.795 0)
+    (property "Footprint" "LED_SMD:LED_0805_2012Metric_Pad1.15x1.40mm_HandSolder" (id 2) (at 100.965 137.795 0)
       (effects (font (size 1.27 1.27)) hide)
     )
@@
       (effects (font (size 1.27 1.27)) (justify left))
     )
-    (property "Footprint" "" (id 2) (at 109.855 62.5602 0)
+    (property "Footprint" "Capacitor_SMD:C_0603_1608Metric_Pad1.08x0.95mm_HandSolder" (id 2) (at 109.855 62.5602 0)
       (effects (font (size 1.27 1.27)) hide)
     )
@@
       (effects (font (size 1.27 1.27)) (justify right))
     )
-    (property "Footprint" "" (id 2) (at 124.46 78.74 0)
+    (property "Footprint" "Connector_PinHeader_2.54mm:PinHeader_1x02_P2.54mm_Vertical" (id 2) (at 124.46 78.74 0)
       (effects (font (size 1.27 1.27)) hide)
     )
@@
       (effects (font (size 1.27 1.27)) (justify right))
     )
-    (property "Footprint" "" (id 2) (at 164.973 103.505 90)
+    (property "Footprint" "Resistor_SMD:R_0603_1608Metric_Pad0.98x0.95mm_HandSolder" (id 2) (at 164.973 103.505 90)
       (effects (font (size 1.27 1.27)) hide)
     )
@@
       (effects (font (size 1.27 1.27)) (justify right))
     )
-    (property "Footprint" "" (id 2) (at 165.608 71.12 90)
+    (property "Footprint" "Resistor_SMD:R_0603_1608Metric_Pad0.98x0.95mm_HandSolder" (id 2) (at 165.608 71.12 90)
       (effects (font (size 1.27 1.27)) hide)
     )
@@
       (effects (font (size 1.27 1.27)) (justify right))
     )
-    (property "Footprint" "" (id 2) (at 164.973 113.665 90)
+    (property "Footprint" "Resistor_SMD:R_0603_1608Metric_Pad0.98x0.95mm_HandSolder" (id 2) (at 164.973 113.665 90)
       (effects (font (size 1.27 1.27)) hide)
     )
@@
       (effects (font (size 1.27 1.27)) (justify left))
     )
-    (property "Footprint" "" (id 2) (at 59.055 49.53 0)
+    (property "Footprint" "Package_TO_SOT_SMD:SOT-23" (id 2) (at 59.055 49.53 0)
       (effects (font (size 1.27 1.27)) (justify left) hide)
     )
@@
     (property "Reference" "R42" (id 0) (at 111.125 86.995 0))
     (property "Value" "499R 0.1% 1/16W" (id 1) (at 111.125 89.535 0))
-    (property "Footprint" "" (id 2) (at 104.267 92.075 90)
+    (property "Footprint" "Capacitor_SMD:C_0402_1005Metric" (id 2) (at 104.267 92.075 90)
       (effects (font (size 1.27 1.27)) hide)
     )
@@
     (property "Reference" "TP1" (id 0) (at 120.65 85.725 90))
     (property "Value" "TestPoint" (id 1) (at 121.92 88.265 90))
-    (property "Footprint" "" (id 2) (at 122.555 86.36 0)
+    (property "Footprint" "TestPoint:TestPoint_Pad_2.0x2.0mm" (id 2) (at 122.555 86.36 0)
       (effects (font (size 1.27 1.27)) hide)
     )
@@
       (effects (font (size 1.27 1.27)) (justify right))
     )
-    (property "Footprint" "" (id 2) (at 98.425 58.293 90)
+    (property "Footprint" "Resistor_SMD:R_0603_1608Metric_Pad0.98x0.95mm_HandSolder" (id 2) (at 98.425 58.293 90)
       (effects (font (size 1.27 1.27)) hide)
     )
@@
       (effects (font (size 1.27 1.27)) (justify right))
     )
-    (property "Footprint" "" (id 2) (at 115.57 114.935 0)
+    (property "Footprint" "Hestia:LVK12R010CER" (id 2) (at 115.57 114.935 0)
       (effects (font (size 1.27 1.27)) hide)
     )
@@
       (effects (font (size 1.27 1.27)) (justify right))
     )
-    (property "Footprint" "" (id 2) (at 165.608 60.96 90)
+    (property "Footprint" "Resistor_SMD:R_0603_1608Metric_Pad0.98x0.95mm_HandSolder" (id 2) (at 165.608 60.96 90)
       (effects (font (size 1.27 1.27)) hide)
     )
@@
       (effects (font (size 1.27 1.27)) (justify left))
     )
-    (property "Footprint" "" (id 2) (at 218.7702 67.945 0)
+    (property "Footprint" "Capacitor_SMD:C_1206_3216Metric" (id 2) (at 218.7702 67.945 0)
       (effects (font (size 1.27 1.27)) hide)
     )
@@
     (property "Reference" "R41" (id 0) (at 103.505 130.175 90))
     (property "Value" "100R 5% 1/10W" (id 1) (at 105.41 129.54 90))
-    (property "Footprint" "" (id 2) (at 99.187 130.175 90)
+    (property "Footprint" "Resistor_SMD:R_0603_1608Metric_Pad0.98x0.95mm_HandSolder" (id 2) (at 99.187 130.175 90)
       (effects (font (size 1.27 1.27)) hide)
     )
@@
       (effects (font (size 1.27 1.27)) (justify left))
     )
-    (property "Footprint" "" (id 2) (at 207.9752 67.945 0)
+    (property "Footprint" "Capacitor_SMD:C_1206_3216Metric" (id 2) (at 207.9752 67.945 0)
       (effects (font (size 1.27 1.27)) hide)
     )
@@
       (effects (font (size 1.27 1.27)) (justify left))
     )
-    (property "Footprint" "" (id 2) (at 229.5652 67.945 0)
+    (property "Footprint" "Capacitor_SMD:C_1206_3216Metric" (id 2) (at 229.5652 67.945 0)
       (effects (font (size 1.27 1.27)) hide)
     )
@@
       (effects (font (size 1.27 1.27)) (justify left))
     )
-    (property "Footprint" "" (id 2) (at 132.08 125.095 0)
+    (property "Footprint" "Package_SO:SOIC-8_3.9x4.9mm_P1.27mm" (id 2) (at 132.08 125.095 0)
       (effects (font (size 1.27 1.27)) (justify left) hide)
     )
@@
     (property "Reference" "FB13" (id 0) (at 123.825 53.975 0))
     (property "Value" "MMZ1608A222BTA00" (id 1) (at 131.445 56.515 0))
-    (property "Footprint" "" (id 2) (at 120.523 55.245 90)
+    (property "Footprint" "Resistor_SMD:R_0603_1608Metric_Pad0.98x0.95mm_HandSolder" (id 2) (at 120.523 55.245 90)
       (effects (font (size 1.27 1.27)) hide)
     )
@@
       (effects (font (size 1.27 1.27)) (justify right))
     )
-    (property "Footprint" "" (id 2) (at 114.173 127.635 90)
-      (effects (font (size 1.27 1.27)) hide)
-    )
+    (property "Footprint" "Resistor_SMD:R_0603_1608Metric_Pad0.98x0.95mm_HandSolder" (id 2) (at 114.173 127.635 90)
+      (effects (font (size 1.27 1.27)) hide)
+    )
