File: hardware/pcb/hestia/PC104.kicad_sch (KiCad schematic)
At the start: 2 parts, among them J3 ESQ-126-39-G-D, J4 ESQ-126-39-G-D

Commit message: exclude J3,J4 from BOM -the pc104 pin sockets. exclude J7,J8,J12,J13,J14,J15,J16 from BOM - the shrouded pin header components for thermistors but we'll probably solder and goop leaded thermistors to the TH footprint pads. SW2 was already set to exclude but is still showing up in BOM. H9 to H17 wire restraint holes were also previously set to exclude in BOM but are still showing up in the BOM.
Parts:
- J3, J4: now left out of the parts list
Changed lines of the file:
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@@
   (no_connect (at 40.64 132.08))
   (symbol (lib_id "Hestia:ESQ-126-39-G-D") (at 64.77 88.9 0) (unit 1)
-    (in_bom yes) (on_board yes)
+    (in_bom no) (on_board yes)
     (property "Reference" "J4" (id 0) (at 62.23 20.32 0)
       (effects (font (size 1.27 1.27)) (justify left))
@@
   )
   (symbol (lib_id "Hestia:ESQ-126-39-G-D") (at 48.26 88.9 0) (unit 1)
-    (in_bom yes) (on_board yes)
+    (in_bom no) (on_board yes)
     (property "Reference" "J3" (id 0) (at 45.72 20.32 0)
       (effects (font (size 1.27 1.27)) (justify left))
