File: hestia-pcb/buck_converter.kicad_sch (KiCad schematic)
At the start: 21 parts, among them U1 LM2655MTC-3.3/NOPB

Commit message: shift template designator/value locations for SRP5030C footprint in library. Update hestia PCB with SRP5030C footprint for L2 on buck regulator. change D7 footprint from SOT23 to smaller SOT-323 as per diode on BOM.
Parts:
- L2: footprint Inductor_SMD:L_Coilcraft_LPS5030 -> Hestia:SRP5030C
Changed lines of the file:
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@@
       (effects (font (size 1.27 1.27)))
     )
-    (property "Footprint" "Inductor_SMD:L_Coilcraft_LPS5030" (at 179.07 90.805 0)
+    (property "Footprint" "Hestia:SRP5030C" (at 179.07 90.805 0)
       (effects (font (size 1.27 1.27)) hide)
     )
