File: hestia-pcb/hestia.kicad_sch (KiCad schematic)
At the start: 76 parts, among them J1 Serial Connector, J2 i2c connector, J5 VREF+, J6 Conn_02x07_Odd_Even, SW1 SW_Push, U2 MSP430F2618TPN_Simplifed, U3 ADS7828, U8 TXB0104PW, U9 LTC4313-1, Y1 32.768kHz 12.5pf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

Commit message: #63: update footprint for LTC4313-1 to match spec
- updated U9 footprint and 3D model
- moved a few pin 1 indicators closer to their chips
- fixed TP5 inconsistency between schematic & pcb
Parts:
- TP5: now left out of the parts list
- U9: footprint Package_DFN_QFN:DFN-8-1EP_3x3mm_P0.65mm_EP1.55x2.4mm -> Package_DFN_QFN:DFN-8-1EP_3x3mm_P0.5mm_EP1.65x2.38mm
Changed lines of the file:
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@@
       (effects (font (size 1.27 1.27)))
     )
-    (property "Footprint" "Package_DFN_QFN:DFN-8-1EP_3x3mm_P0.65mm_EP1.55x2.4mm" (at 233.68 140.97 0)
-      (effects (font (size 1.27 1.27)) hide)
-    )
-    (property "Datasheet" "" (at 233.68 140.97 0)
+    (property "Footprint" "Package_DFN_QFN:DFN-8-1EP_3x3mm_P0.5mm_EP1.65x2.38mm" (at 233.68 140.97 0)
+      (effects (font (size 1.27 1.27)) hide)
+    )
+    (property "Datasheet" "https://www.analog.com/media/en/technical-documentation/data-sheets/4313123f.pdf" (at 233.68 140.97 0)
       (effects (font (size 1.27 1.27)) hide)
     )
@@
   )
   (symbol (lib_id "Connector:TestPoint") (at 259.715 154.305 0) (unit 1)
-    (in_bom yes) (on_board yes) (dnp no)
+    (in_bom no) (on_board yes) (dnp no)
     (property "Reference" "TP5" (at 260.985 151.765 0)
       (effects (font (size 1.27 1.27)) (justify left))
